File: ECM_Preamp/ECM_Preamp.kicad_sch (KiCad schematic)
At the start: 23 parts, among them J1 Conn_Coaxial, J2 XLR3, Q1 BF245C, SW1 SW_DIP_x02

Commit message: sim updated, C_pol updated
Parts:
- C5: value C_Polarized -> (none); footprint Capacitor_THT:CP_Radial_D5.0mm_P2.50mm -> (none)
Changed lines of the file:
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@@
     (in_bom yes) (on_board yes) (fields_autoplaced)
     (property "Reference" "C5" (id 0) (at 136.271 73.8845 90))
-    (property "Value" "C_Polarized" (id 1) (at 136.271 76.6596 90))
-    (property "Footprint" "Capacitor_THT:CP_Radial_D5.0mm_P2.50mm" (id 2) (at 140.97 79.0448 0)
+    (property "Value" "" (id 1) (at 136.271 76.6596 90))
+    (property "Footprint" "" (id 2) (at 140.97 79.0448 0)
       (effects (font (size 1.27 1.27)) hide)
     )
@@
     )
     (path "/91d9e0c9-862b-4f86-9074-ebe4bfc5ae13"
-      (reference "C5") (unit 1) (value "C_Polarized") (footprint "Capacitor_THT:CP_Radial_D5.0mm_P2.50mm")
+      (reference "C5") (unit 1) (value "1000u/35V") (footprint "Capacitor_THT:CP_Radial_D13.0mm_P5.00mm")
     )
     (path "/9f22985d-999b-44f5-9bb3-64c9181b6668"

Commit message: Updated component values
Parts:
- C2, C6: value C_Polarized -> (none); footprint Capacitor_THT:CP_Radial_D5.0mm_P2.50mm -> (none)
- C5: value (none) -> 1000u/35V; footprint (none) -> Capacitor_THT:CP_Radial_D13.0mm_P5.00mm
- D1, D4: value D_Zener -> (none); footprint Diode_THT:D_A-405_P7.62mm_Horizontal -> (none)
- D2, D3: value D -> (none); footprint Diode_THT:D_T-1_P5.08mm_Horizontal -> (none)
- R1: value 5.1k -> 5.6k
- R3: value 5.1k -> 10k
- R6: value 6.8k -> 100R
Other:
- note added: "8.2V"
- note added: "Load ~33kOhm"
Changed lines of the file:
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@@
     (stroke (width 0) (type default) (color 0 0 0 0))
+  )
+  (text "Load ~33kOhm" (at 19.05 90.17 0)
+    (effects (font (size 1.27 1.27)) (justify left bottom))
+  )
+  (text "8.2V" (at 48.26 49.53 0)
+    (effects (font (size 1.27 1.27)) (justify left bottom))
   )
   (label "P48" (at 201.93 63.5 0)
@@
       (effects (font (size 1.27 1.27)) (justify left))
     )
-    (property "Value" "D_Zener" (id 1) (at 61.722 60.2866 90)
-      (effects (font (size 1.27 1.27)) (justify left))
-    )
-    (property "Footprint" "Diode_THT:D_A-405_P7.62mm_Horizontal" (id 2) (at 59.69 58.42 0)
+    (property "Value" "" (id 1) (at 61.722 60.2866 90)
+      (effects (font (size 1.27 1.27)) (justify left))
+    )
+    (property "Footprint" "" (id 2) (at 59.69 58.42 0)
       (effects (font (size 1.27 1.27)) hide)
     )
@@
     (in_bom yes) (on_board yes) (fields_autoplaced)
     (property "Reference" "R6" (id 0) (at 176.53 45.8175 90))
-    (property "Value" "6.8k" (id 1) (at 176.53 48.5926 90))
+    (property "Value" "100R" (id 1) (at 176.53 48.5926 90))
     (property "Footprint" "Resistor_THT:R_Axial_DIN0204_L3.6mm_D1.6mm_P7.62mm_Horizontal" (id 2) (at 176.53 52.578 90)
       (effects (font (size 1.27 1.27)) hide)
@@
       (effects (font (size 1.27 1.27)) (justify left))
     )
-    (property "Value" "D" (id 1) (at 69.342 95.8466 90)
-      (effects (font (size 1.27 1.27)) (justify left))
-    )
-    (property "Footprint" "Diode_THT:D_T-1_P5.08mm_Horizontal" (id 2) (at 67.31 93.98 0)
+    (property "Value" "" (id 1) (at 69.342 95.8466 90)
+      (effects (font (size 1.27 1.27)) (justify left))
+    )
+    (property "Footprint" "" (id 2) (at 67.31 93.98 0)
       (effects (font (size 1.27 1.27)) hide)
     )
@@
     (in_bom yes) (on_board yes) (fields_autoplaced)
     (property "Reference" "C5" (id 0) (at 136.271 73.8845 90))
-    (property "Value" "" (id 1) (at 136.271 76.6596 90))
-    (property "Footprint" "" (id 2) (at 140.97 79.0448 0)
+    (property "Value" "1000u/35V" (id 1) (at 136.271 76.6596 90))
+    (property "Footprint" "Capacitor_THT:CP_Radial_D13.0mm_P5.00mm" (id 2) (at 140.97 79.0448 0)
       (effects (font (size 1.27 1.27)) hide)
     )
@@
       (effects (font (size 1.27 1.27)) (justify right))
     )
-    (property "Value" "5.1k" (id 1) (at 48.768 72.9866 0)
+    (property "Value" "5.6k" (id 1) (at 48.768 72.9866 0)
       (effects (font (size 1.27 1.27)) (justify right))
     )
@@
       (effects (font (size 1.27 1.27)) (justify left))
     )
-    (property "Value" "C_Polarized" (id 1) (at 79.121 59.3976 0)
-      (effects (font (size 1.27 1.27)) (justify left))
-    )
-    (property "Footprint" "Capacitor_THT:CP_Radial_D5.0mm_P2.50mm" (id 2) (at 77.1652 62.23 0)
+    (property "Value" "" (id 1) (at 79.121 59.3976 0)
+      (effects (font (size 1.27 1.27)) (justify left))
+    )
+    (property "Footprint" "" (id 2) (at 77.1652 62.23 0)
       (effects (font (size 1.27 1.27)) hide)
     )
@@
       (effects (font (size 1.27 1.27)) (justify left))
     )
-    (property "Value" "D_Zener" (id 1) (at 162.052 59.0166 90)
-      (effects (font (size 1.27 1.27)) (justify left))
-    )
-    (property "Footprint" "Diode_THT:D_A-405_P7.62mm_Horizontal" (id 2) (at 160.02 57.15 0)
+    (property "Value" "" (id 1) (at 162.052 59.0166 90)
+      (effects (font (size 1.27 1.27)) (justify left))
+    )
+    (property "Footprint" "" (id 2) (at 160.02 57.15 0)
       (effects (font (size 1.27 1.27)) hide)
     )
@@
       (effects (font (size 1.27 1.27)) (justify left))
     )
-    (property "Value" "C_Polarized" (id 1) (at 146.431 58.1276 0)
-      (effects (font (size 1.27 1.27)) (justify left))
-    )
-    (property "Footprint" "Capacitor_THT:CP_Radial_D5.0mm_P2.50mm" (id 2) (at 144.4752 60.96 0)
+    (property "Value" "" (id 1) (at 146.431 58.1276 0)
+      (effects (font (size 1.27 1.27)) (justify left))
+    )
+    (property "Footprint" "" (id 2) (at 144.4752 60.96 0)
       (effects (font (size 1.27 1.27)) hide)
     )
@@
     (in_bom yes) (on_board yes) (fields_autoplaced)
     (property "Reference" "R3" (id 0) (at 91.44 45.8175 90))
-    (property "Value" "5.1k" (id 1) (at 91.44 48.5926 90))
+    (property "Value" "10k" (id 1) (at 91.44 48.5926 90))
     (property "Footprint" "Resistor_THT:R_Axial_DIN0204_L3.6mm_D1.6mm_P7.62mm_Horizontal" (id 2) (at 91.44 49.022 90)
       (effects (font (size 1.27 1.27)) hide)
@@
       (effects (font (size 1.27 1.27)) (justify left))
     )
-    (property "Value" "D" (id 1) (at 69.342 80.489 90)
-      (effects (font (size 1.27 1.27)) (justify left))
-    )
-    (property "Footprint" "Diode_THT:D_T-1_P5.08mm_Horizontal" (id 2) (at 69.342 83.2641 90)
+    (property "Value" "" (id 1) (at 69.342 80.489 90)
+      (effects (font (size 1.27 1.27)) (justify left))
+    )
+    (property "Footprint" "" (id 2) (at 69.342 83.2641 90)
       (effects (font (size 1.27 1.27)) (justify left))
     )
@@
     )
     (path "/9dd0c413-39dc-4212-a3af-ed4348a5474b"
-      (reference "C2") (unit 1) (value "C_Polarized") (footprint "Capacitor_THT:CP_Radial_D5.0mm_P2.50mm")
+      (reference "C2") (unit 1) (value "100u/25V") (footprint "Capacitor_THT:CP_Radial_D5.0mm_P2.50mm")
     )
     (path "/0344fcc0-1bce-4826-a842-99a1bbab53e5"
@@
     )
     (path "/9f22985d-999b-44f5-9bb3-64c9181b6668"
-      (reference "C6") (unit 1) (value "C_Polarized") (footprint "Capacitor_THT:CP_Radial_D5.0mm_P2.50mm")
+      (reference "C6") (unit 1) (value "47u/35V") (footprint "Capacitor_THT:CP_Radial_D5.0mm_P2.50mm")
     )
     (path "/160960bd-7577-4b21-8cf3-a3b5ab725215"
-      (reference "D1") (unit 1) (value "D_Zener") (footprint "Diode_THT:D_A-405_P7.62mm_Horizontal")
+      (reference "D1") (unit 1) (value "8,2V") (footprint "Diode_THT:D_A-405_P7.62mm_Horizontal")
     )
     (path "/d1cd8821-9f7e-4a19-bc27-523ccf34cb3f"
-      (reference "D2") (unit 1) (value "D") (footprint "Diode_THT:D_T-1_P5.08mm_Horizontal")
+      (reference "D2") (unit 1) (value "1N4148") (footprint "Diode_THT:D_T-1_P5.08mm_Horizontal")
     )
     (path "/8e469742-f87d-41c4-a512-12e581ec31a4"
-      (reference "D3") (unit 1) (value "D") (footprint "Diode_THT:D_T-1_P5.08mm_Horizontal")
+      (reference "D3") (unit 1) (value "1N4148") (footprint "Diode_THT:D_T-1_P5.08mm_Horizontal")
     )
     (path "/9f02238d-3eec-42d9-bf87-229dc16888e2"
-      (reference "D4") (unit 1) (value "D_Zener") (footprint "Diode_THT:D_A-405_P7.62mm_Horizontal")
+      (reference "D4") (unit 1) (value "18V") (footprint "Diode_THT:D_A-405_P7.62mm_Horizontal")
     )
     (path "/eaa94493-19fb-4bcb-a9e6-69dae981540d"
@@
     )
     (path "/94344474-bec1-4e32-b6d4-4c1cb78f3c65"
-      (reference "R1") (unit 1) (value "5.1k") (footprint "Resistor_THT:R_Axial_DIN0204_L3.6mm_D1.6mm_P7.62mm_Horizontal")
+      (reference "R1") (unit 1) (value "5.6k") (footprint "Resistor_THT:R_Axial_DIN0204_L3.6mm_D1.6mm_P7.62mm_Horizontal")
     )
     (path "/9f4f01da-a7a3-4151-8036-0e878c9dfb62"
@@
     )
     (path "/bec17670-6719-4af0-986c-64e6627a19b3"
-      (reference "R3") (unit 1) (value "5.1k") (footprint "Resistor_THT:R_Axial_DIN0204_L3.6mm_D1.6mm_P7.62mm_Horizontal")
+      (reference "R3") (unit 1) (value "10k") (footprint "Resistor_THT:R_Axial_DIN0204_L3.6mm_D1.6mm_P7.62mm_Horizontal")
     )
     (path "/9f47dca3-2f71-4dfa-92b5-7c8fd16eb772"
@@
     )
     (path "/7eac98fe-2d1d-4293-89c6-65aeb4beea5d"
-      (reference "R6") (unit 1) (value "6.8k") (footprint "Resistor_THT:R_Axial_DIN0204_L3.6mm_D1.6mm_P7.62mm_Horizontal")
+      (reference "R6") (unit 1) (value "100R") (footprint "Resistor_THT:R_Axial_DIN0204_L3.6mm_D1.6mm_P7.62mm_Horizontal")
     )
     (path "/49fff740-7847-43e9-af01-20faa22d2671"
